File: LAMPU_EMERGENCY_v1.3_all_module_smd/LAMPU_EMERGENCY_v1.3_all_module_smd.sch (EAGLE design)
At the start: 62 parts, among them Q1 IRF540D2PACK, T1 SS8050, T4 SS8050, T5 SS8050, T6 SS8050, T8 SS8050, X1 BATTERY_1, X2 AC_PIN, X3 MOSOUT, X4 BATTERY2, X6 MOSOUT, X7 AC_PIN

Commit message: Split X and Y vibration sensors
separate it, maybe someone use sensors have different type
Parts:
- SL1: value VIBRATION_X -> VIBRATION_Y
- SL3: value VIBRATION_Y -> VIBRATION_X
Connections:
- removed net VIB_SEN: SL1.2, SL3.2, U$2.A2
- new net VIB_SEN_X: SL3.2, U$2.A2
- new net VIB_SEN_Y: SL1.2, U$2.A1
Other:
- moved on the sheet: C1, SV1
